File: ddkb.kicad_pcb (KiCad board)
At the start: 2 copper layers, 257.2 x 76.2 mm, 117 parts, among them J1 Conn_01x04, J2 Conn_01x02, J3 Conn_01x03, J4 MX-NoLED, K1 MX-NoLED, M1 MX-NoLED, P1 MX-NoLED, Q1 MX-NoLED, SW1 SW_Push, T1 MX-NoLED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

Commit message: small reroutes
Parts:
- moved C1 4.38 mm to (32.5, 78.8), turned to 0 degrees
- moved C7 1.73 mm to (51.2, 77.0), turned to 45 degrees
- moved C8 1.21 mm to (48.5, 78.8), turned to 135 degrees
- moved C12 0.78 mm to (46.0, 81.2), turned to 135 degrees
- moved R4 0.63 mm to (44.6, 91.8)
- moved C16 0.63 mm to (45.4, 92.6)
- moved Y1 0.63 mm to (47.9, 93.4)
- moved C15 0.63 mm to (47.1, 90.9)
- moved C10 0.59 mm to (56.0, 85.8), turned to -45 degrees
- moved C5 0.56 mm to (52.0, 77.8), turned to 45 degrees
- moved C11 0.51 mm to (49.2, 78.0)
- moved C14 0.29 mm to (53.2, 88.8)
- moved C3 0.27 mm to (45.2, 87.5)
- moved C13 0.25 mm to (46.0, 88.2)
- moved C4 0.22 mm to (55.0, 79.5)
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Routing:
- net +3.3V: track 130.7 -> 126.9 mm
- net COL1: track 96.0 -> 98.0 mm
- net GND: track 33.7 -> 32.1 mm, vias 19 -> 20
- net /XIN: track 10.2 -> 8.84 mm
- net COL4: track 126.7 -> 125.9 mm
- net COL2: track 88.6 -> 87.8 mm
- net COL3: track 87.5 -> 86.7 mm
- net ROW2: track 251.7 -> 252.4 mm
- net /XOUT: track 6.69 -> 6.02 mm
- net ROW3: track 229.0 -> 229.7 mm

Commit message: indrease jst marigin
Parts:
- removed J2: Conn_01x02, Button_Switch_SMD:SW_SPST_CK_RS282G05A3
- added SW2: SW_Push, Button_Switch_SMD:SW_SPST_TL3342, B.Cu at (74.0, 73.0)
- moved R3 7.26 mm to (67.8, 73.5)
- moved C2 6.78 mm to (31.9, 69.9)
- moved J1 6.40 mm to (36.5, 72.1)
- moved U2 5.36 mm to (27.7, 73.4)
- moved J3 4.13 mm to (38.4, 91.1)
- moved C1 2.21 mm to (30.3, 78.5), turned to 180 degrees
- moved C17 0.70 mm to (62.5, 69.4)
- moved C7 0.62 mm to (51.1, 77.6)
- moved C5 0.59 mm to (51.8, 78.3)
Routing:
- net +3.3V: track 126.9 -> 137.3 mm
- net ROW0: track 288.9 -> 297.2 mm
- net /QSPI_SS: track 26.6 -> 19.0 mm
- net /USB_D-: track 13.6 -> 19.7 mm
- net /USB_D+: track 13.6 -> 19.7 mm
- net /~{USB_BOOT}: track 3.86 -> 9.86 mm
- net /SWCLK: track 15.3 -> 11.0 mm
- net /SWD: track 20.1 -> 15.9 mm
- net VCOM: track 7.69 -> 5.40 mm
- net GND: track 32.1 -> 34.0 mm, vias 20 -> 16

Commit message: add second bottom row
Parts:
- added REF**: 1.25U, ddkb:MX-1.25U-NoLED, F.Cu at (208.8, 120.6)
- added REF**: 1.5U, ddkb:MX-1.5U-NoLED, F.Cu at (82.5, 120.6)
- added REF**: 5.25U, ddkb:MX-1U-NoLED, F.Cu at (146.8, 120.6)
- moved D11 5.38 mm to (91.6, 123.0)
- moved /1 1.83 mm to (244.5, 101.5)
- moved ;1 1.83 mm to (234.9, 82.5)
- moved B1 1.83 mm to (149.2, 101.5)
- moved D25 1.83 mm to (181.0, 65.8)
- moved D28 1.83 mm to (181.0, 123.0)
- moved D32 1.83 mm to (219.1, 65.8)
- moved D35 1.83 mm to (219.1, 123.0)
- moved G1 1.83 mm to (139.7, 82.5)
- moved K1 1.83 mm to (196.8, 82.5)
- moved M1 1.83 mm to (187.3, 101.5)
- moved O1 1.83 mm to (211.1, 63.4)
- moved U4 1.83 mm to (173.0, 63.4)
- moved A1 1.83 mm to (63.5, 82.5)
- moved C10 1.83 mm to (55.2, 84.1)
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Routing:
- net Net-(D18-A): track 8.05 -> 40.6 mm
- net COL4: track 125.9 -> 156.2 mm
- net COL2: track 87.8 -> 99.5 mm
- net Net-(D11-A): track 8.05 -> 14.6 mm
- net Net-(D35-A): track 8.05 -> 10.5 mm
Other:
- outline, holes or cut-outs redrawn

Commit message: small adjustment
Routing:
- net ROW1: track 283.5 -> 297.0 mm
Changed lines of the file:
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@@
   (segment (start 227.965 96.4575) (end 233.3625 101.855) (width 0.2) (layer "B.Cu") (net 9))
   (segment (start 233.3625 101.855) (end 233.3625 102.26875) (width 0.2) (layer "B.Cu") (net 9))
-  (segment (start 44.80625 55.75) (end 37.80625 62.75) (width 0.2) (layer "F.Cu") (net 10))
-  (segment (start 71.20625 63.75) (end 63.20625 55.75) (width 0.2) (layer "F.Cu") (net 10))
-  (segment (start 63.20625 55.75) (end 44.80625 55.75) (width 0.2) (layer "F.Cu") (net 10))
+  (segment (start 35.71875 56.35625) (end 62.70625 56.35625) (width 0.2) (layer "F.Cu") (net 10))
+  (segment (start 34.925 59.53125) (end 34.925 57.15) (width 0.2) (layer "F.Cu") (net 10))
+  (segment (start 32.13325 62.323) (end 34.925 59.53125) (width 0.2) (layer "F.Cu") (net 10))
+  (segment (start 34.925 57.15) (end 35.71875 56.35625) (width 0.2) (layer "F.Cu") (net 10))
+  (segment (start 71.20625 64.85625) (end 71.20625 65.0875) (width 0.2) (layer "F.Cu") (net 10))
+  (segment (start 33.3375 75.40625) (end 32.13325 74.202) (width 0.2) (layer "F.Cu") (net 10))
+  (segment (start 41.8625 75.40625) (end 33.3375 75.40625) (width 0.2) (layer "F.Cu") (net 10))
+  (segment (start 42.80625 76.35) (end 41.8625 75.40625) (width 0.2) (layer "F.Cu") (net 10))
+  (segment (start 32.13325 74.202) (end 32.13325 62.323) (width 0.2) (layer "F.Cu") (net 10))
+  (segment (start 62.70625 56.35625) (end 71.20625 64.85625) (width 0.2) (layer "F.Cu") (net 10))
   (segment (start 74.00625 86.55) (end 74.00625 75.75) (width 0.2) (layer "F.Cu") (net 10))
-  (segment (start 71.20625 72.95) (end 71.20625 63.75) (width 0.2) (layer "F.Cu") (net 10))
-  (segment (start 37.80625 71.35) (end 42.80625 76.35) (width 0.2) (layer "F.Cu") (net 10))
   (segment (start 74.00625 75.75) (end 71.20625 72.95) (width 0.2) (layer "F.Cu") (net 10))
-  (segment (start 37.80625 62.75) (end 37.80625 71.35) (width 0.2) (layer "F.Cu") (net 10))
+  (segment (start 71.20625 72.95) (end 71.20625 65.0875) (width 0.2) (layer "F.Cu") (net 10))
   (via (at 42.80625 76.35) (size 0.6) (drill 0.3) (layers "F.Cu" "B.Cu") (net 10))
   (via (at 74.00625 86.55) (size 0.6) (drill 0.3) (layers "F.Cu" "B.Cu") (net 10))
@@
   (segment (start 55.20625 72.6) (end 55.20625 69.6) (width 0.2) (layer "B.Cu") (net 85))
   (segment (start 56.95625 67.85) (end 57.854275 67.85) (width 0.2) (layer "B.Cu") (net 85))
+  (segment (start 52.687907 80.763927) (end 56.204864 77.246971) (width 0.2) (layer "B.Cu") (net 86))
   (segment (start 56.204864 73.032928) (end 55.60625 72.434314) (width 0.2) (layer "B.Cu") (net 86))
-  (segment (start 56.739093 68.632843) (end 56.841068 68.632843) (width 0.2) (layer "B.Cu") (net 86))
+  (segment (start 55.60625 72.434314) (end 55.60625 69.765686) (width 0.2) (layer "B.Cu") (net 86))
   (segment (start 56.204864 77.246971) (end 56.204864 73.032928) (width 0.2) (layer "B.Cu") (net 86))
-  (segment (start 56.841068 68.632843) (end 57.711653 69.503428) (width 0.2) (layer "B.Cu") (net 86))
-  (segment (start 55.60625 72.434314) (end 55.60625 69.765686) (width 0.2) (layer "B.Cu") (net 86))
-  (segment (start 52.687907 80.763927) (end 56.204864 77.246971) (width 0.2) (layer "B.Cu") (net 86))
-  (segment (start 55.60625 69.765686) (end 56.739093 68.632843) (width 0.2) (layer "B.Cu") (net 86))
+  (segment (start 55.60625 69.765686) (end 56.315686 69.05625) (width 0.2) (layer "B.Cu") (net 86))
+  (segment (start 57.264475 69.05625) (end 57.711653 69.503428) (width 0.2) (layer "B.Cu") (net 86))
+  (segment (start 56.315686 69.05625) (end 57.264475 69.05625) (width 0.2) (layer "B.Cu") (net 86))
   (segment (start 57.662173 71.25) (end 56.813627 70.401454) (width 0.2) (layer "B.Cu") (net 87))
   (segment (start 52.97075 81.04677) (end 57.662173 76.355347) (width 0.2) (layer "B.Cu") (net 87))

Commit message: add split left shift
Parts:
- added REF**: 1.25U, ddkb:MX-1.25U-NoLED, F.Cu at (32.5, 101.5)
Routing:
- net Net-(D3-A): track 13.4 -> 23.9 mm
- net COL0: track 62.5 -> 70.0 mm
- net GND: track 34.0 -> 38.8 mm, vias 16 -> 17
- net COL1: track 98.0 -> 96.5 mm
- net Net-(D11-A): track 14.6 -> 13.6 mm
