File: ddkb.kicad_pcb (KiCad board)
At the start: 2 copper layers, 257.2 x 76.2 mm, 121 parts, among them J1 Conn_01x04, J3 Conn_01x03, J4 MX-NoLED, K1 MX-NoLED, M1 MX-NoLED, P1 MX-NoLED, Q1 MX-NoLED, SW1 SW_Push, SW2 SW_Push, T1 MX-NoLED, U1 RP2040, U2 NCP1117-3.3_SOT223, U3 W25Q128JVS, U4 MX-NoLED, X1 MX-NoLED, Y1 YSX321SL, Y2 MX-NoLED

Commit message: change ldo
Parts:
- removed U2: NCP1117-3.3_SOT223, Package_TO_SOT_SMD:SOT-223-3_TabPin2
- added U5: XC6206P332MR, Package_TO_SOT_SMD:SOT-23-3, B.Cu at (29.0, 71.1)
- C1, C2: value 10u -> 1u
- moved C1 5.35 mm to (26.7, 72.3), turned to -90 degrees
- moved C2 4.74 mm to (26.7, 70.0)
Routing:
- net GND: track 38.8 -> 45.5 mm, vias 17 -> 18
- net ROW0: track 297.2 -> 290.6 mm
- net VCOM: track 5.40 -> 7.70 mm
- net +3.3V: track 136.8 -> 137.8 mm

Commit message: add qspi_ss pullup
Parts:
- added R5: 10k, Resistor_SMD:R_0402_1005Metric, B.Cu at (67.0, 70.8)
- moved C16 1.10 mm to (60.9, 67.0)
- moved C2 0.26 mm to (54.0, 78.0)
- moved C4 0.25 mm to (53.3, 77.3)
- renumbered C3 to C1, C13 to C10, C14 to C11, C1 to C12, C15 to C13, C16 to C14, C2 to C15, C17 to C16, C18 to C17, C4 to C2, C5 to C3, C6 to C4, C7 to C5, C8 to C6, C10 to C7, C11 to C8, C12 to C9, D45 to D15, D15 to D16, D16 to D17, D17 to D18, D18 to D19, D19 to D20, D20 to D21, D21 to D22, D22 to D23, D23 to D24, D24 to D25, D25 to D26, D26 to D27, D27 to D28, D28 to D29, D29 to D30, D30 to D31, D31 to D32, D32 to D33, D33 to D34, D34 to D35, D35 to D36, D36 to D37, D37 to D38, D38 to D39, D39 to D40, D40 to D41, D41 to D42, D42 to D43, D43 to D44, D44 to D45, J3 to J2, J4 to J3, R5 to R6, R6 to R7, SW2 to SW1, SW1 to SW2, U5 to U2
Connections:
- D19 pad 2: Net-(D18-A) -> Net-(D19-A)
- D36 pad 2: Net-(D35-A) -> Net-(D36-A)
- LSPACE1 pad 2: Net-(D18-A) -> Net-(D19-A)
- RGUI1 pad 2: Net-(D35-A) -> Net-(D36-A)
Routing:
- net +3.3V: track 137.8 -> 144.5 mm
- net GND: track 45.5 -> 44.4 mm

Commit message: cleanup
Connections:
- REF** pad 2: Net-(D35-A) -> Net-(D36-A)
- REF** pad 2: Net-(D18-A) -> Net-(D19-A)
Routing:
- net Net-(D18-A): track 40.6 -> 0.00 mm
- net Net-(D19-A): track 0.00 -> 40.4 mm
- net Net-(D35-A): track 10.5 -> 0.00 mm
- net Net-(D36-A): track 0.00 -> 10.4 mm
- net GND: track 44.4 -> 46.7 mm, vias 18 -> 19
- net /QSPI_SS: track 19.0 -> 20.4 mm
